File: resources/KiCad/RingTheBell/3.3V.kicad_sch (KiCad schematic)
At the start: 6 parts, among them SW7 SW_SPST, SW8 SW_SPST

Commit message: tighten up the schematics
Connections:
- net at A8. (3V3): now also R12.1
- net at A9.~ (IO1_09): now also LS4.2; no longer A8. (3V3)
- net at A9.~ (IO1_09), SW7.1 (A), SW8.1 (A): no longer A8. (3V3)
- new net: A8. (3V3), A9.~ (IO1_09) (x3)
Other:
- moved on the sheet: A9A, LS4, R12
