File: resources/KiCad/RingTheBell/3.3V_UART.kicad_sch (KiCad schematic)
At the start: 10 parts, among them SW1 SW_SPST, SW2 SW_SPST

Commit message: tighten up the schematics
Connections:
- net at A4. (3V3), R2.2, R4.2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: no longer A3.~ (IO1_09)
- net at A4. (3V3): now also A3.~ (IO1_09)
- net at A3.~ (IO1_09): no longer A4. (3V3)
Other:
- moved on the sheet: A3A, LS1, R5

Commit message: tighten up the schematics
Connections:
- net at A4. (3V3), R2.2, R4.2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: now also A3.~ (IO1_09)
- net at A4. (3V3): now also A3.~ (IO1_09)
- net at A3.~ (IO1_09): no longer A4. (3V3)
Changed lines of the file:
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@@
+	)
+	(junction
+		(at 104.14 168.91)
+		(diameter 0)
+		(color 0 0 0 0)
 	)
 	(junction
@@
 	(wire
 		(pts
+			(xy 104.14 168.91) (xy 113.03 168.91)
+		)
+		(stroke
+			(width 0)
+			(type default)
+		)
+	)
+	(wire
+		(pts
 			(xy 133.35 168.91) (xy 133.35 133.35)
 		)
@@
 	(wire
 		(pts
-			(xy 29.21 168.91) (xy 113.03 168.91)
-		)
-		(stroke
+			(xy 104.14 149.86) (xy 104.14 168.91)
+		)
+		(stroke
+			(width 0)
+			(type default)
+		)
+	)
+	(wire
+		(pts
+			(xy 29.21 168.91) (xy 104.14 168.91)
+		)
+		(stroke
