File: resources/KiCad/RingTheBell/74HCT125N.kicad_sch (KiCad schematic)
At the start: 11 parts, among them SW5 SW_SPST, SW6 SW_SPST

Commit message: tighten up the schematics
Connections:
- net at A5. (3V3), A6.~ (IO1_09), A7.~ (3Y_08)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: no longer R10.1
- net at A6.~ (IO1_09): now also R7.2
- net at A5. (3V3): now also SW5.2 (B)
- net at A7.~ (3Y_08): now also R7.1; no longer A5. (3V3)
- new net: A6.~ (IO1_09), R10.1
- new net: A5. (3V3), A6.~ (IO1_09), A7.~ (3Y_08)
- new net: A5. (3V3), A7.~ (3Y_08)
Other:
- moved on the sheet: A6A, LS3, R7

Commit message: tighten up the schematics
Connections:
- net at A6.~ (IO1_09): now also R7.2
- net at A5. (3V3): now also SW5.2 (B)
- net at A7.~ (3Y_08): now also R7.1; no longer A5. (3V3)
- new net: A5. (3V3), A6.~ (IO1_09), A7.~ (3Y_08)
- new net: A5. (3V3), A7.~ (3Y_08)
Other:
- moved on the sheet: A6A, LS3, R7
Changed lines of the file:
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@@
 	(text "Yellow"
 		(exclude_from_sim no)
-		(at 122.936 137.16 0)
+		(at 122.936 130.048 0)
 		(effects
 			(font
@@
 	(text "Yellow"
 		(exclude_from_sim no)
-		(at 102.616 143.764 0)
+		(at 104.14 133.35 0)
 		(effects
 			(font
@@
 	(text "Blue"
 		(exclude_from_sim no)
-		(at 64.77 138.684 0)
+		(at 64.77 141.224 0)
 		(effects
 			(font
@@
 	(text "Green"
 		(exclude_from_sim no)
-		(at 65.024 136.398 0)
+		(at 65.024 138.938 0)
 		(effects
 			(font
@@
 	(wire
 		(pts
-			(xy 104.14 149.86) (xy 104.14 165.1)
+			(xy 104.14 152.4) (xy 104.14 165.1)
 		)
 		(stroke
@@
 	(wire
 		(pts
-			(xy 45.72 139.7) (xy 45.72 118.11)
+			(xy 50.8 115.57) (xy 133.35 115.57)
 		)
 		(stroke
@@
 	(wire
 		(pts
-			(xy 99.06 144.78) (xy 123.19 144.78)
+			(xy 54.61 154.94) (xy 68.58 154.94)
 		)
 		(stroke
@@
 	(wire
 		(pts
-			(xy 50.8 115.57) (xy 133.35 115.57)
+			(xy 52.07 139.7) (xy 50.8 139.7)
 		)
 		(stroke
@@
 	(wire
 		(pts
-			(xy 54.61 152.4) (xy 68.58 152.4)
+			(xy 50.8 115.57) (xy 50.8 139.7)
 		)
 		(stroke
@@
 	(wire
 		(pts
-			(xy 52.07 137.16) (xy 50.8 137.16)
+			(xy 113.03 165.1) (xy 128.27 165.1)
 		)
 		(stroke
@@
 	(wire
 		(pts
-			(xy 113.03 165.1) (xy 128.27 165.1)
+			(xy 128.27 127) (xy 128.27 129.54)
 		)
 		(stroke
@@
 	(wire
 		(pts
-			(xy 128.27 127) (xy 128.27 129.54)
+			(xy 31.75 83.82) (xy 29.21 83.82)
 		)
 		(stroke
@@
 	(wire
 		(pts
-			(xy 31.75 83.82) (xy 29.21 83.82)
+			(xy 58.42 99.06) (xy 29.21 99.06)
 		)
 		(stroke
@@
 	(wire
 		(pts
-			(xy 58.42 99.06) (xy 29.21 99.06)
+			(xy 128.27 134.62) (xy 128.27 165.1)
 		)
 		(stroke
@@
 	(wire
 		(pts
-			(xy 128.27 134.62) (xy 128.27 165.1)
+			(xy 147.32 82.55) (xy 133.35 82.55)
 		)
 		(stroke
@@
 	(wire
 		(pts
-			(xy 147.32 82.55) (xy 133.35 82.55)
+			(xy 58.42 102.87) (xy 58.42 110.49)
 		)
 		(stroke
@@
 	(wire
 		(pts
-			(xy 58.42 102.87) (xy 58.42 110.49)
+			(xy 99.06 137.16) (xy 123.19 137.16)
 		)
 		(stroke
@@
 	(wire
 		(pts
-			(xy 58.42 110.49) (xy 58.42 134.62)
+			(xy 147.32 77.47) (xy 140.97 77.47)
 		)
 		(stroke
@@
 	(wire
 		(pts
-			(xy 147.32 77.47) (xy 140.97 77.47)
+			(xy 123.19 137.16) (xy 123.19 118.11)
 		)
 		(stroke
@@
 	(wire
 		(pts
-			(xy 68.58 139.7) (xy 45.72 139.7)
+			(xy 68.58 142.24) (xy 45.72 142.24)
 		)
 		(stroke
@@
 	(wire
 		(pts
-			(xy 57.15 137.16) (xy 68.58 137.16)
+			(xy 57.15 139.7) (xy 68.58 139.7)
 		)
 		(stroke
@@
 	(wire
 		(pts
-			(xy 99.06 149.86) (xy 104.14 149.86)
+			(xy 99.06 152.4) (xy 104.14 152.4)
 		)
 		(stroke
@@
 	(wire
 		(pts
-			(xy 104.14 165.1) (xy 113.03 165.1)
+			(xy 45.72 118.11) (xy 45.72 142.24)
 		)
 		(stroke
@@
 	(wire
 		(pts
-			(xy 50.8 137.16) (xy 50.8 115.57)
+			(xy 104.14 165.1) (xy 113.03 165.1)
 		)
 		(stroke
@@
 	(wire
 		(pts
-			(xy 58.42 134.62) (xy 68.58 134.62)
+			(xy 58.42 137.16) (xy 68.58 137.16)
 		)
 		(stroke
@@
 	(wire
 		(pts
-			(xy 54.61 149.86) (xy 57.15 149.86)
+			(xy 54.61 152.4) (xy 57.15 152.4)
 		)
 		(stroke
@@
 	(wire
 		(pts
-			(xy 123.19 144.78) (xy 123.19 118.11)
+			(xy 181.61 77.47) (xy 181.61 110.49)
 		)
 		(stroke
@@
 	(wire
 		(pts
-			(xy 181.61 77.47) (xy 181.61 110.49)
+			(xy 57.15 149.86) (xy 68.58 149.86)
 		)
 		(stroke
@@
 	(wire
 		(pts
-			(xy 57.15 147.32) (xy 68.58 147.32)
+			(xy 181.61 77.47) (xy 177.8 77.47)
 		)
 		(stroke
@@
 	(wire
 		(pts
-			(xy 181.61 77.47) (xy 177.8 77.47)
+			(xy 45.72 118.11) (xy 113.03 118.11)
 		)
 		(stroke
@@
 	(wire
 		(pts
-			(xy 45.72 118.11) (xy 113.03 118.11)
+			(xy 137.16 49.53) (xy 137.16 127)
 		)
 		(stroke
@@
 	(wire
 		(pts
-			(xy 137.16 49.53) (xy 137.16 127)
+			(xy 113.03 134.62) (xy 113.03 165.1)
 		)
 		(stroke
@@
 	(wire
 		(pts
-			(xy 113.03 134.62) (xy 113.03 165.1)
+			(xy 58.42 110.49) (xy 58.42 137.16)
 		)
 		(stroke
@@
 	(wire
 		(pts
-			(xy 57.15 149.86) (xy 57.15 147.32)
+			(xy 57.15 152.4) (xy 57.15 149.86)
 		)
 		(stroke
@@
 	(symbol
 		(lib_id "Device:Speaker")
-		(at 49.53 149.86 0)
+		(at 49.53 152.4 0)
 		(mirror y)
 		(unit 1)
@@
 		(dnp no)
 		(property "Reference" "LS3"
-			(at 44.45 149.8599 0)
+			(at 44.45 152.3999 0)
 			(effects
 				(font
@@
 		)
 		(property "Value" "Speaker"
-			(at 44.45 152.3999 0)
+			(at 44.45 154.9399 0)
 			(effects
 				(font
@@
 		)
 		(property "Footprint" ""
-			(at 49.53 154.94 0)
+			(at 49.53 157.48 0)
 			(effects
 				(font
@@
 		)
 		(property "Datasheet" "~"
-			(at 49.784 151.13 0)
+			(at 49.784 153.67 0)
 			(effects
 				(font
@@
 		)
 		(property "Description" "Speaker"
-			(at 49.53 149.86 0)
+			(at 49.53 152.4 0)
 			(effects
 				(font
@@
 		(lib_name "YX5200_1")
 		(lib_id "mdoLibrary:YX5200")
-		(at 83.82 152.4 0)
+		(at 83.82 154.94 0)
 		(unit 1)
 		(exclude_from_sim no)
@@
 		(fields_autoplaced yes)
 		(property "Reference" "A6"
-			(at 83.82 128.27 0)
+			(at 83.82 130.81 0)
 			(effects
 				(font
@@
 		)
 		(property "Value" "YX5200"
-			(at 83.82 130.81 0)
+			(at 83.82 133.35 0)
 			(effects
 				(font
@@
 		)
 		(property "Footprint" ""
-			(at 83.82 152.4 0)
+			(at 83.82 154.94 0)
 			(effects
 				(font
@@
 		)
 		(property "Datasheet" ""
-			(at 83.82 152.4 0)
+			(at 83.82 154.94 0)
 			(effects
 				(font
@@
 		)
 		(property "Description" ""
-			(at 83.82 152.4 0)
+			(at 83.82 154.94 0)
 			(effects
 				(font
@@
 	(symbol
 		(lib_id "Device:R_Small_US")
-		(at 54.61 137.16 90)
+		(at 54.61 139.7 90)
 		(unit 1)
 		(exclude_from_sim no)
@@
 		(dnp no)
 		(property "Reference" "R7"
-			(at 54.864 130.81 90)
+			(at 54.864 133.35 90)
 			(effects
 				(font
@@
 		)
 		(property "Value" "1K"
-			(at 54.864 133.858 90)
+			(at 54.864 136.398 90)
 			(effects
 				(font
@@
 		)
 		(property "Footprint" ""
-			(at 54.61 137.16 0)
+			(at 54.61 139.7 0)
 			(effects
 				(font
@@
 		)
 		(property "Datasheet" "~"
-			(at 54.61 137.16 0)
+			(at 54.61 139.7 0)
 			(effects
 				(font
@@
 		)
 		(property "Description" "Resistor, small US symbol"
-			(at 54.61 137.16 0)
+			(at 54.61 139.7 0)
 			(effects
 				(font
